Commit message: Added docking logic

File: install/psolar_gazebo/share/psolar_gazebo/urdf/turtlebot3_waffle_pi.urdf (robot description, URDF)
Before this commit: robot turtlebot3_waffle_pi, 8 links, 7 joints
Links:
- added link camera_link; collision box size=0.015 0.030 0.027
- added link camera_rgb_frame
- added link camera_rgb_optical_frame
Joints:
- added joint camera_joint: type fixed, parent base_link, child camera_link, origin xyz=0.073 -0.011 0.084 rpy=0 0 0
- added joint camera_rgb_joint: type fixed, parent camera_link, child camera_rgb_frame, origin xyz=0.003 0.011 0.009 rpy=0 0 0
- added joint camera_rgb_optical_joint: type fixed, parent camera_rgb_frame, child camera_rgb_optical_frame, origin xyz=0 0 0 rpy=-1.57 0 -1.57
